Commit message: fix：Taks_T1

File: resources/robots/Taks_T1/urdf/Taks_T1/Taks_T1.urdf (robot description, URDF)
Before this commit: robot Taks_T1, 33 links, 32 joints
Links:
- link left_ankle_roll_link: geometry collision mesh filename=meshes/left_ankle_roll_link.STL; visual mesh filename=meshes/left_ankle_roll_link.STL
- link right_ankle_roll_link: geometry collision mesh filename=meshes/right_ankle_roll_link.STL; visual mesh filename=meshes/right_ankle_roll_link.STL
Joints:
- joint left_ankle_pitch_joint: limit lower=-0.87267 upper=0.5236 effort=27.0 velocity=3.77 -> lower=-0.87267 upper=0.5236 effort=27.0 velocity=5.4454
- joint left_ankle_roll_joint: limit lower=-0.2618 upper=0.2618 effort=27.0 velocity=3.77 -> lower=-0.2618 upper=0.2618 effort=27.0 velocity=5.4454
- joint left_elbow_joint: limit lower=-0.7 upper=1.57 effort=27.0 velocity=3.77 -> lower=-0.7 upper=1.57 effort=27.0 velocity=5.4454
- joint left_hip_pitch_joint: origin xyz=0.115 0.0 -0.0523 rpy=0.0 0.0 -1.5707963267948966 -> xyz=0.0 0.115 -0.0523 rpy=0 0 0
- joint left_shoulder_pitch_joint: limit lower=-3.0 upper=2.0 effort=27.0 velocity=3.77 -> lower=-3.0 upper=2.0 effort=27.0 velocity=5.4454
- joint left_shoulder_roll_joint: limit lower=-0.2 upper=2.2515 effort=27.0 velocity=3.77 -> lower=-0.2 upper=2.2515 effort=27.0 velocity=5.4454
- joint left_shoulder_yaw_joint: limit lower=-2.58 upper=2.58 effort=27.0 velocity=3.77 -> lower=-2.58 upper=2.58 effort=27.0 velocity=5.4454
- joint left_wrist_pitch_joint: limit lower=-0.9 upper=0.9 effort=7.0 velocity=12.57 -> lower=-0.9 upper=0.9 effort=7.0 velocity=20.944
- joint left_wrist_roll_joint: limit lower=-2.67 upper=2.67 effort=7.0 velocity=12.57 -> lower=-2.67 upper=2.67 effort=7.0 velocity=20.944
- joint left_wrist_yaw_joint: limit lower=-0.9 upper=0.9 effort=7.0 velocity=12.57 -> lower=-0.9 upper=0.9 effort=7.0 velocity=20.944
- joint right_ankle_pitch_joint: limit lower=-0.87267 upper=0.5236 effort=27.0 velocity=3.77 -> lower=-0.87267 upper=0.5236 effort=27.0 velocity=5.4454
- joint right_ankle_roll_joint: limit lower=-0.2618 upper=0.2618 effort=27.0 velocity=3.77 -> lower=-0.2618 upper=0.2618 effort=27.0 velocity=5.4454
- joint right_elbow_joint: limit lower=-0.7 upper=1.57 effort=27.0 velocity=3.77 -> lower=-0.7 upper=1.57 effort=27.0 velocity=5.4454
- joint right_hip_pitch_joint: origin xyz=-0.115 0.0 -0.0523 rpy=0.0 0.0 -1.5707963267948966 -> xyz=0.0 -0.115 -0.0523 rpy=0 0 0
- joint right_shoulder_pitch_joint: limit lower=-2.0 upper=2.0 effort=27.0 velocity=3.77 -> lower=-2.0 upper=2.0 effort=27.0 velocity=5.4454
- joint right_shoulder_roll_joint: limit lower=-2.2515 upper=0.2 effort=27.0 velocity=3.77 -> lower=-2.2515 upper=0.2 effort=27.0 velocity=5.4454
- joint right_shoulder_yaw_joint: limit lower=-2.58 upper=2.58 effort=27.0 velocity=3.77 -> lower=-2.58 upper=2.58 effort=27.0 velocity=5.4454
- joint right_wrist_pitch_joint: limit lower=-0.9 upper=0.9 effort=7.0 velocity=12.57 -> lower=-0.9 upper=0.9 effort=7.0 velocity=20.944
- joint right_wrist_roll_joint: limit lower=-2.67 upper=2.67 effort=7.0 velocity=12.57 -> lower=-2.67 upper=2.67 effort=7.0 velocity=20.944
- joint right_wrist_yaw_joint: limit lower=-0.9 upper=0.9 effort=7.0 velocity=12.57 -> lower=-0.9 upper=0.9 effort=7.0 velocity=20.944
- joint waist_yaw_joint: origin xyz=0.0 0.0 0.0 rpy=0.0 0.0 -1.5707963267948966 -> xyz=0.0 0.0 0.0 rpy=0 0 0
